File: BTS7960_controller_shield.kicad_pcb (KiCad board)
At the start: 4 copper layers, 100.4 x 48 mm, 63 parts, among them J1 Conn_ST_STDC14, J2 Conn_02x04_Odd_Even, J3 USB_C_Receptacle_USB2.0, J4 Conn_01x04, J5 USB_C_Receptacle_USB2.0, Q1 BTN8982TA, Q2 BTN8982TA, U1 LDFM33PVR, U2 STM32F302K8Ux, U3 USBLC6-2SC6, Y1 16MHz

Commit message: New idea
Parts:
- removed the C1 at (119.0, 154.5)
- removed the C1 at (97.5, 144.4)
- removed the C2 at (123.8, 154.5)
- removed the C2 at (97.5, 139.6)
- removed the C7 at (124.3, 152.5)
- removed the C7 at (95.5, 139.1)
- removed the C8 at (118.8, 152.0)
- removed the C8 at (95.0, 144.6)
- removed the C9 at (124.8, 144.6)
- removed the C9 at (87.6, 138.6)
- removed the D1 at (127.2, 129.3)
- removed the D1 at (74.8, 139.1)
- removed the D3 at (127.1, 147.0)
- removed the D3 at (90.8, 135.1)
- removed the H1 at (122.4, 120.0)
- removed the H1 at (70.0, 120.0)
- removed the H2 at (162.4, 160.0)
- removed the H2 at (110.0, 160.0)
- removed the H3 at (162.4, 120.0)
- removed the H3 at (110.0, 120.0)
- removed the H4 at (122.4, 160.0)
- removed the H4 at (70.0, 160.0)
- removed the J2 at (148.2, 161.5)
- removed the J2 at (95.8, 161.5)
- removed the J3 at (121.5, 133.0)
- removed the J3 at (69.1, 142.7)
- removed the J4 at (143.6, 160.1)
- removed the J4 at (110.5, 131.6)
- removed the J5 at (135.4, 161.0)
- removed the J5 at (111.0, 147.0)
- removed JP1 (x2): SolderJumper_3_Open, Jumper:SolderJumper-3_P2.0mm_Open_TrianglePad1.0x1.5mm_NumberLabels
- removed Q1, Q2: BTN8982TA, Package_TO_SOT_SMD:TO-263-7_TabPin8
- removed the R1 at (126.9, 127.0)
- removed the R1 at (74.5, 136.8)
- removed the R2 at (118.7, 150.2)
- removed the R2 at (93.2, 144.7)
- removed the R4 at (127.1, 149.9)
- removed the R4 at (93.7, 135.1)
- removed the R5 at (128.7, 146.9)
- removed the R5 at (100.8, 140.0)
- removed R6 (x2), R7 (x2), R8 (x2): 10k, Resistor_SMD:R_0402_1005Metric_Pad0.72x0.64mm_HandSolder
- removed the REF** at (134.5, 130.5)
- removed the REF** at (162.4, 132.5)
- removed the U2 at (122.4, 148.2)
- removed the U2 at (91.2, 141.0)
- removed the U3 at (128.4, 133.0)
- removed the U3 at (76.0, 142.8)
- removed the Y1 at (121.4, 154.1)
- removed the Y1 at (97.1, 142.0)
- added C1: 12pF, Capacitor_SMD:C_0402_1005Metric_Pad0.74x0.62mm_HandSolder, F.Cu at (80.2, 132.5)
- added C10: 0.1uF, Capacitor_SMD:C_0402_1005Metric_Pad0.74x0.62mm_HandSolder, F.Cu at (75.8, 140.3)
- added C11: 1uF, Capacitor_SMD:C_0402_1005Metric_Pad0.74x0.62mm_HandSolder, F.Cu at (83.5, 130.5)
- added C12: 10nF, Capacitor_SMD:C_0402_1005Metric_Pad0.74x0.62mm_HandSolder, F.Cu at (76.0, 138.3)
- added C13: 0.1uF, Capacitor_SMD:C_0402_1005Metric_Pad0.74x0.62mm_HandSolder, F.Cu at (87.8, 127.4)
- added C14: 0.1uF, Capacitor_SMD:C_0402_1005Metric_Pad0.74x0.62mm_HandSolder, F.Cu at (80.2, 134.5)
- added C2: 12pF, Capacitor_SMD:C_0402_1005Metric_Pad0.74x0.62mm_HandSolder, F.Cu at (79.2, 136.4)
- added C6: 2.2uF, Capacitor_SMD:C_0402_1005Metric_Pad0.74x0.62mm_HandSolder, F.Cu at (76.0, 136.4)
- added C7: 0.1uF, Capacitor_SMD:C_0402_1005Metric_Pad0.74x0.62mm_HandSolder, F.Cu at (72.8, 138.3)
- added C8: 0.1uF, Capacitor_SMD:C_0402_1005Metric_Pad0.74x0.62mm_HandSolder, F.Cu at (88.3, 125.4)
- added C9: 0.1uF, Capacitor_SMD:C_0402_1005Metric_Pad0.74x0.62mm_HandSolder, F.Cu at (72.6, 140.3)
- added D1: Red, LED_SMD:LED_0603_1608Metric_Pad1.05x0.95mm_HandSolder, F.Cu at (60.5, 139.6)
- added D3: Red, LED_SMD:LED_0603_1608Metric_Pad1.05x0.95mm_HandSolder, F.Cu at (60.5, 137.0)
- added H1: MountingHole, MountingHole:MountingHole_3.2mm_M3, F.Cu at (17.0, 153.0)
- added H2: MountingHole, MountingHole:MountingHole_3.2mm_M3, F.Cu at (57.0, 153.0)
- added H3: MountingHole, MountingHole:MountingHole_3.2mm_M3, F.Cu at (17.0, 193.0)
- added H4: MountingHole, MountingHole:MountingHole_3.2mm_M3, F.Cu at (57.0, 193.0)
- added J2: Conn_02x04_Odd_Even, Connector_PinSocket_2.54mm:PinSocket_2x04_P2.54mm_Vertical, B.Cu at (18.5, 167.2)
- added J3: USB_C_Receptacle_USB2.0, Connector_USB:USB_C_Receptacle_XKB_U262-16XN-4BVC11, F.Cu at (37.0, 152.5)
- added J4: Conn_02x04_Odd_Even, Connector_PinSocket_2.54mm:PinSocket_2x04_P2.54mm_Vertical, B.Cu at (55.5, 178.8)
- added J5: Conn_01x05, Connector_JST:JST_PH_S5B-PH-K_1x05_P2.00mm_Horizontal, F.Cu at (26.0, 190.0)
- added J6: Conn_01x05, Connector_JST:JST_PH_S5B-PH-K_1x05_P2.00mm_Horizontal, F.Cu at (40.0, 190.0)
- added L1: 39nH, Inductor_SMD:L_0603_1608Metric, F.Cu at (47.4, 116.7)
- added R1: 1k5, Resistor_SMD:R_0402_1005Metric_Pad0.72x0.64mm_HandSolder, F.Cu at (85.1, 125.4)
- added R2: 10k, Resistor_SMD:R_0402_1005Metric_Pad0.72x0.64mm_HandSolder, F.Cu at (72.8, 136.4)
- added R4: 10k, Resistor_SMD:R_0402_1005Metric_Pad0.72x0.64mm_HandSolder, F.Cu at (84.6, 127.9)
- added R5: 1k5, Resistor_SMD:R_0402_1005Metric_Pad0.72x0.64mm_HandSolder, F.Cu at (64.3, 141.0)
- added REF**: OSHW-Logo2_9.8x8mm_SilkScreen, Symbol:OSHW-Logo2_9.8x8mm_SilkScreen, B.Cu at (37.0, 173.0)
- added RN1: R_Pack03, Package_DIP:DIP-6_W8.89mm_SMDSocket_LongPads, F.Cu at (66.1, 100.8)
- added RN2: R_Pack03, Package_DIP:DIP-6_W8.89mm_SMDSocket_LongPads, F.Cu at (66.1, 110.2)
- added SW1: SW_SPST, Button_Switch_THT:SW_Tactile_SPST_Angled_PTS645Vx58-2LFS, F.Cu at (23.5, 151.8)
- added SW2: SW_SPST, Button_Switch_THT:SW_Tactile_SPST_Angled_PTS645Vx58-2LFS, F.Cu at (46.0, 151.8)
- added U2: STM32F411CEUx, Package_DFN_QFN:QFN-48-1EP_7x7mm_P0.5mm_EP5.6x5.6mm, F.Cu at (36.9, 173.0)
- added U3: USBLC6-2SC6, Package_TO_SOT_SMD:SOT-23-6, F.Cu at (37.0, 160.0)
- added Y1: 16MHz, Crystal:Crystal_SMD_Abracon_ABM10-4Pin_2.5x2.0mm, F.Cu at (36.4, 179.6)
- moved J1 56.2 mm to (29.0, 164.0), turned to 270 degrees
- moved C4 13.6 mm to (81.3, 125.7), turned to 0 degrees
- moved U1 12.7 mm to (68.9, 139.7), turned to 0 degrees
- moved D2 11.4 mm to (77.0, 125.7)
- moved C5 10.8 mm to (80.8, 128.3), turned to 0 degrees
- moved C3 10.5 mm to (69.0, 136.6), turned to 0 degrees
- moved R3 6.04 mm to (80.2, 130.5), turned to 0 degrees
Connections:
- J1 pad 10: (no net) -> JTDI
- J1 pad 13: USART1_TX -> (no net)
- J1 pad 14: USART1_RX -> (no net)
Routing:
- net (no net): track 147.8 -> 0.00 mm, vias 21 -> 0
- net VBUS: track 49.9 -> 0.00 mm
- net Net-(J4-Pad1): track 34.8 -> 0.00 mm, vias 3 -> 0
- net PWM_H: track 32.5 -> 0.00 mm, vias 2 -> 0
- net DIR_B: track 31.1 -> 0.00 mm, vias 1 -> 0
- net ENC_B: track 29.8 -> 0.00 mm, vias 4 -> 0
- net DIR_A: track 29.6 -> 0.00 mm, vias 1 -> 0
- net ~RST: track 25.4 -> 0.00 mm, vias 2 -> 0
- net ENC_A: track 25.3 -> 0.00 mm
- net SWDIO: track 19.7 -> 0.00 mm
- net USART1_TX: track 19.7 -> 0.00 mm, vias 2 -> 0
- net +3V3: track 18.9 -> 0.00 mm, vias 9 -> 0
- net SWCLK: track 18.0 -> 0.00 mm
- net SWO: track 17.2 -> 0.00 mm
- net USART1_RX: track 16.5 -> 0.00 mm
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- removed copper zone on B.Cu, net (none)
- removed copper zone on F.Cu, net (none)
- removed copper zone on In1.Cu, net (none)
- removed copper zone on In2.Cu, net (none)
- removed copper zone on F.Cu, net +3V3
- removed copper zone on In2.Cu, net +3V3
- removed copper zone on B.Cu, net GND
- removed copper zone on F.Cu, net GND
- removed copper zone on In1.Cu, net GND
Other:
- board size 100.4 x 48 mm -> 48 x 48 mm
- board text removed: "+"
- board text removed: "-"
- board text removed: "3V3"
- board text removed: "3V3 -> 0R"
- board text removed: "5V"
- board text removed: "A"
- board text removed: "B"
- board text removed: "BTS7960 MODULE CONTROLLER"
- board text removed: "ENCODER"
- board text removed: "TO HOST"
- board text removed: "USB"
- board text removed: "WARNING! CUSTOM USB"

Commit message: Przygotowanie do projektu
Parts:
- removed C1, C2: 12pF, Capacitor_SMD:C_0402_1005Metric_Pad0.74x0.62mm_HandSolder
- removed C10, C13, C14, C7, C8, C9: 0.1uF, Capacitor_SMD:C_0402_1005Metric_Pad0.74x0.62mm_HandSolder
- removed C11: 1uF, Capacitor_SMD:C_0402_1005Metric_Pad0.74x0.62mm_HandSolder
- removed C12: 10nF, Capacitor_SMD:C_0402_1005Metric_Pad0.74x0.62mm_HandSolder
- removed C3, C4: 10uF, Capacitor_SMD:C_0603_1608Metric_Pad1.08x0.95mm_HandSolder
- removed C5: 1uF, Capacitor_SMD:C_0603_1608Metric_Pad1.08x0.95mm_HandSolder
- removed C6: 2.2uF, Capacitor_SMD:C_0402_1005Metric_Pad0.74x0.62mm_HandSolder
- removed D1, D2, D3: Red, LED_SMD:LED_0603_1608Metric_Pad1.05x0.95mm_HandSolder
- removed H1, H2, H3, H4: MountingHole, MountingHole:MountingHole_3.2mm_M3
- removed J1: Conn_ST_STDC14, Connector_PinHeader_1.27mm:PinHeader_2x07_P1.27mm_Vertical_SMD
- removed J3: USB_C_Receptacle_USB2.0, Connector_USB:USB_C_Receptacle_XKB_U262-16XN-4BVC11
- removed J5, J6: Conn_01x05, Connector_JST:JST_PH_S5B-PH-K_1x05_P2.00mm_Horizontal
- removed L1: 39nH, Inductor_SMD:L_0603_1608Metric
- removed R1, R5: 1k5, Resistor_SMD:R_0402_1005Metric_Pad0.72x0.64mm_HandSolder
- removed R2, R4: 10k, Resistor_SMD:R_0402_1005Metric_Pad0.72x0.64mm_HandSolder
- removed R3: 650, Resistor_SMD:R_0402_1005Metric_Pad0.72x0.64mm_HandSolder
- removed REF**: OSHW-Logo2_9.8x8mm_SilkScreen, Symbol:OSHW-Logo2_9.8x8mm_SilkScreen
- removed RN1, RN2: R_Pack03, Package_DIP:DIP-6_W8.89mm_SMDSocket_LongPads
- removed SW1, SW2: SW_SPST, Button_Switch_THT:SW_Tactile_SPST_Angled_PTS645Vx58-2LFS
- removed U1: LDFM33PVR, Package_DFN_QFN:DFN-6-1EP_2x2mm_P0.5mm_EP0.61x1.42mm
- removed U2: STM32F411CEUx, Package_DFN_QFN:QFN-48-1EP_7x7mm_P0.5mm_EP5.6x5.6mm
- removed U3: USBLC6-2SC6, Package_TO_SOT_SMD:SOT-23-6
- removed Y1: 16MHz, Crystal:Crystal_SMD_Abracon_ABM10-4Pin_2.5x2.0mm
- moved J2 13.0 mm to (21.0, 180.0), turned to 90 degrees
- moved J4 5.18 mm to (60.5, 180.0), turned to 90 degrees
Other:
- board size 48 x 48 mm -> 51 x 20 mm
